File: Eagle files/openSipPuff (rev C).sch (EAGLE design)
At the start: 20 parts, among them J2 1X04-RA, J3 AVR_SPI_PRG_62X3_LOCK, U1 ATMEGA32U4TQFP, U2 AD8223, U3 MPX12GP, Y1 16MHz

Commit message: Rev C updates
New Eagle files and BOM.
Parts:
- removed CN1: (no value), adafruit:USBMOLEX
- added CN2: (no value), adafruit:USBMINIB
- added LED2: RED, led:LEDCHIPLED_0805
- added LED3: BLUE, led:LEDCHIPLED_0805
- added R6, R7: 82, SparkFun-Resistors:RESISTOR0805-RES
- added SENSOR, SENSOR1: (no value), SparkFun-Connectors:M04PTH
- J2: value 1X04-RA -> I2C; device sip-and-puff:1X04-RA -> SparkFun-Connectors:M04PTH
- LOGO1: value OSHW-LOGOM -> OSHW-LOGOL; device SparkFun-Aesthetics:OSHW-LOGOM -> SparkFun-Aesthetics:OSHW-LOGOL
- Y1: device SparkFun-FreqCtrl:RESONATORPTH -> SparkFun-FreqCtrl:RESONATOR16MHZ
- renumbered J3 to J1
Connections:
- removed net SENSOR_OUT: U1.PF0(ADC0), U2.VOUT
- new net N$14: LED3.A, R7.2
- new net N$15: LED2.A, R6.2
- new net N$8: R6.1, U1.PF1(ADC1)
- new net N$9: R7.1, U1.PF0(ADC0)
- new net OUTPUT: U1.PF4(ADC4), U2.VOUT
- new net SCL: J2.4, U1.PD0(SCL)
- new net SDA: J2.3, U1.PD1(SDA)
- net 5V: now also J2.1, SENSOR.3, SENSOR1.3; no longer J2.3
- net D+: now also CN2.D+; no longer CN1.D+
- net D-: now also CN2.D-; no longer CN1.D-
- net GND: now also CN2.GND, J2.2, LED2.C, LED3.C, SENSOR.1, SENSOR1.1; no longer CN1.GND, J2.1
- net N$10: now also SENSOR.2, SENSOR1.2; no longer J2.2
- net N$13: now also SENSOR.4, SENSOR1.4; no longer J2.4
- net N$4: now also CN2.VBUS; no longer CN1.VBUS
Other:
- moved on the sheet: R5
